File: jlink-st-adapter.kicad_pcb (KiCad board)
At the start: 2 copper layers, 35.6 x 27.9 mm, 5 parts, among them J1 STDC14, J2 J-Link, J3 Mode Jumper, J4 Mode Jumper, J5 Serial Header

Commit message: New files and updates for KiCad 6.0
Connections:
- net /~RST renamed /~{RST}
- J1 pad 1: Net-(J1-Pad1) -> unconnected-(J1-Pad1)
- J1 pad 11: Net-(J1-Pad11) -> unconnected-(J1-Pad11)
- J1 pad 2: Net-(J1-Pad2) -> unconnected-(J1-Pad2)
- J2 pad 14: Net-(J2-Pad14) -> unconnected-(J2-Pad14)
- J2 pad 16: Net-(J2-Pad16) -> unconnected-(J2-Pad16)
- J2 pad 18: Net-(J2-Pad18) -> unconnected-(J2-Pad18)
- J2 pad 2: Net-(J2-Pad2) -> unconnected-(J2-Pad2)
- J2 pad 20: Net-(J2-Pad20) -> unconnected-(J2-Pad20)
- J2 pad 3: Net-(J2-Pad3) -> unconnected-(J2-Pad3)
- J4 pad 3: Net-(J4-Pad3) -> unconnected-(J4-Pad3)
Other:
- net class Default removed
